File: switching_regulator_2.kicad_sch (KiCad schematic)
At the start: 11 parts, among them IC1 ST1S41PHR, J1 TBL009-254-04GY-2GY, J2 TBL009-254-04GY-2GY, J3 571-0100, J4 571-0500

Commit message: [ADD] curved tracks
Parts:
- R1, R2: now not fitted
Changed lines of the file:
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@@
 		(in_bom yes)
 		(on_board yes)
-		(dnp no)
+		(dnp yes)
 		(fields_autoplaced yes)
 		(property "Reference" "R2"
@@
 		(in_bom yes)
 		(on_board yes)
-		(dnp no)
+		(dnp yes)
 		(property "Reference" "R1"
 			(at 182.88 63.4999 90)
